File: Motherboard 2024/Motherboard 2024.kicad_pcb (KiCad board)
At the start: 2 copper layers, 212 x 189 mm, 76 parts, among them J1 43650-0221, J10 Conn_01x02, J11 43650-0221, J12 43650-0221, J13 43650-0221, J14 Conn_01x02, J15 Conn_01x02, J16 43650-0221, J17 43650-0221, J18 43650-0221, J19 43650-0221, J2 43650-0221, J24 ECU_A, J25 ECU_B, J26 43650-0221, J27 43045-1015, J3 43650-0221, J34 HW-08-XX-XX-D-XXX-SM, J35 HW-08-XX-XX-D-XXX-SM, J36 HW-08-XX-XX-D-XXX-SM, J37 HW-08-XX-XX-D-XXX-SM, J38 BSPD_TEST_SWITCH, J39 SHOULDER_RESET, J40 AIR_POWER, J41 TSMS_IN, J42 GLV_MASTER_SWITCH_OUT, J43 GLV_MASTER_SWITCH_OUT, J44 24V_BATTERY+, J45 24V_BATTERY+, J6 43650-0221, J7 43650-0221, J8 43650-0221, J9 Conn_01x02

Commit message: Updated 12 Sep
Parts:
- moved J45 17.9 mm to (191.9, 45.3)
- moved J44 10.6 mm to (212.9, 45.3)
- moved J43 10.2 mm to (202.0, 60.1)
- moved MAIN_RELAY_CONROL1 8.00 mm to (230.3, 42.0)
- moved 24_BATTERY+ 6.86 mm to (216.9, 52.8)
- moved J42 5.16 mm to (201.8, 74.9)
- renumbered 24_BATTERY+1 to 24_BATTERY+, AIR_POWER1 to AIR_POWER, BSPD_TEST_SWITCH1 to BSPD_TEST_SWITCH, ECU_5V1 to ECU_5V, ECU_ACCEL_SIG2 to ECU_ACCEL_SIG, ECU_ACCEL_SIG1 to ECU_ACCEL_SIG, ECU_BRAKE_INPUT2 to ECU_BRAKE_INPUT, ECU_BRAKE_INPUT1 to ECU_BRAKE_INPUT, GLV_MASTER_SWITCH_OUT1 to GLV_MASTER_SWITCH_OUT, MASTER_ACC_BSPD_CT1 to MASTER_ACC_BSPD_CT, MC_OK_INDICATOR1 to MC_OK_INDICATOR, MOTOR_CONTROLLER_ON_SIG1 to MOTOR_CONTROLLER_ON_SIG, PRECHARGE_CONTROL1 to PRECHARGE_CONTROL, PUMP_ON_SIG1 to PUMP_ON_SIG, RADIATOR_FAN_ON_SIG1 to RADIATOR_FAN_ON_SIG, SHOULDER_RESET1 to SHOULDER_RESET, TSAL_GREEN1 to TSAL_GREEN, TSAL_RED1 to TSAL_RED, TSMS_IN1 to TSMS_IN
Routing:
- net /MAIN_RELAY_CONTROL: track 315.0 -> 322.1 mm
- net /24V_BATTERY+: track 7.86 -> 11.6 mm, vias 4 -> 3
- net /GLV_MASTER_SWITCH_OUT: track 15.4 -> 18.1 mm
