File: Motherboard 2024/Motherboard 2024.kicad_sch (KiCad schematic)
At the start: 76 parts, among them J1 43650-0221, J10 Conn_01x02, J11 43650-0221, J12 43650-0221, J13 43650-0221, J14 Conn_01x02, J15 Conn_01x02, J16 43650-0221, J17 43650-0221, J18 43650-0221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

Commit message: Updated 12 Sep
Parts:
- renumbered PRES_1 to BREAK_PRESSED1
